Commit message: drone fully fixed - getting map now

File: src/ve_behaviours/urdf/x3.gazebo.xacro (robot description, xacro)
@@ -1,131 +1,311 @@
 <?xml version="1.0"?>
 <robot name="X3" xmlns:xacro="http://www.ros.org/wiki/xacro">
-  <!-- Visual toggles -->
-  <xacro:arg name="laser_visual"  default="false"/>
-  <xacro:arg name="camera_visual" default="false"/>
-  <xacro:arg name="depth_visual"  default="false"/>
-  <xacro:arg name="imu_visual"    default="false"/>
-  <!-- Motors & velocity control (unchanged) -->
-  <!-- ... your four MulticopterMotorModel plugins here ... -->
-  <gazebo>
-    <plugin filename="libignition-gazebo-multicopter-control-system.so"
+    <xacro:arg name="laser_visual" default="false" />
+    <xacro:arg name="camera_visual" default="false" />
+    <xacro:arg name="imu_visual" default="false" />
+    <xacro:arg name="depth_visual"  default="false"/>
+    <!-- Quadcopter rotor and velocity control -->
+    <gazebo>
+        <plugin name="ignition::gazebo::systems::MulticopterMotorModel"
+            filename="libignition-gazebo-multicopter-motor-model-system.so">
+            <robotNamespace>X3</robotNamespace>
+            <jointName>rotor_0_joint</jointName>
+            <linkName>rotor_0</linkName>
+            <turningDirection>ccw</turningDirection>
+            <timeConstantUp>0.0125</timeConstantUp>
+            <timeConstantDown>0.025</timeConstantDown>
+            <maxRotVelocity>800.0</maxRotVelocity>
+            <motorConstant>8.54858e-06</motorConstant>
+            <momentConstant>0.016</momentConstant>
+            <commandSubTopic>gazebo/command/motor_speed</commandSubTopic>
+            <motorNumber>0</motorNumber>
+            <rotorDragCoefficient>8.06428e-05</rotorDragCoefficient>
+            <rollingMomentCoefficient>1e-06</rollingMomentCoefficient>
+            <motorSpeedPubTopic>motor_speed/0</motorSpeedPubTopic>
+            <rotorVelocitySlowdownSim>10</rotorVelocitySlowdownSim>
+            <motorType>velocity</motorType>
+        </plugin>
+        <plugin name="ignition::gazebo::systems::MulticopterMotorModel"
+            filename="libignition-gazebo-multicopter-motor-model-system.so">
+            <robotNamespace>X3</robotNamespace>
+            <jointName>rotor_1_joint</jointName>
+            <linkName>rotor_1</linkName>
+            <turningDirection>ccw</turningDirection>
+            <timeConstantUp>0.0125</timeConstantUp>
+            <timeConstantDown>0.025</timeConstantDown>
+            <maxRotVelocity>800.0</maxRotVelocity>
+            <motorConstant>8.54858e-06</motorConstant>
+            <momentConstant>0.016</momentConstant>
+            <commandSubTopic>gazebo/command/motor_speed</commandSubTopic>
+            <motorNumber>1</motorNumber>
+            <rotorDragCoefficient>8.06428e-05</rotorDragCoefficient>
+            <rollingMomentCoefficient>1e-06</rollingMomentCoefficient>
+            <motorSpeedPubTopic>motor_speed/1</motorSpeedPubTopic>
+            <rotorVelocitySlowdownSim>10</rotorVelocitySlowdownSim>
+            <motorType>velocity</motorType>
+        </plugin>
+        <plugin name="ignition::gazebo::systems::MulticopterMotorModel"
+            filename="libignition-gazebo-multicopter-motor-model-system.so">
+            <robotNamespace>X3</robotNamespace>
+            <jointName>rotor_2_joint</jointName>
+            <linkName>rotor_2</linkName>
+            <turningDirection>cw</turningDirection>
+            <timeConstantUp>0.0125</timeConstantUp>
+            <timeConstantDown>0.025</timeConstantDown>
+            <maxRotVelocity>800.0</maxRotVelocity>
+            <motorConstant>8.54858e-06</motorConstant>
+            <momentConstant>0.016</momentConstant>
+            <commandSubTopic>gazebo/command/motor_speed</commandSubTopic>
+            <motorNumber>2</motorNumber>
+            <rotorDragCoefficient>8.06428e-05</rotorDragCoefficient>
+            <rollingMomentCoefficient>1e-06</rollingMomentCoefficient>
+            <motorSpeedPubTopic>motor_speed/2</motorSpeedPubTopic>
+            <rotorVelocitySlowdownSim>10</rotorVelocitySlowdownSim>
+            <motorType>velocity</motorType>
+        </plugin>
+        <plugin name="ignition::gazebo::systems::MulticopterMotorModel"
+            filename="libignition-gazebo-multicopter-motor-model-system.so">
+            <robotNamespace>X3</robotNamespace>
+            <jointName>rotor_3_joint</jointName>
+            <linkName>rotor_3</linkName>
+            <turningDirection>cw</turningDirection>
+            <timeConstantUp>0.0125</timeConstantUp>
+            <timeConstantDown>0.025</timeConstantDown>
+            <maxRotVelocity>800.0</maxRotVelocity>
+            <motorConstant>8.54858e-06</motorConstant>
+            <momentConstant>0.016</momentConstant>
+            <commandSubTopic>gazebo/command/motor_speed</commandSubTopic>
+            <motorNumber>3</motorNumber>
+            <rotorDragCoefficient>8.06428e-05</rotorDragCoefficient>
+            <rollingMomentCoefficient>1e-06</rollingMomentCoefficient>
+            <motorSpeedPubTopic>motor_speed/3</motorSpeedPubTopic>
+            <rotorVelocitySlowdownSim>10</rotorVelocitySlowdownSim>
+            <motorType>velocity</motorType>
+        </plugin>
+        <!-- Quadcopter velocity control -->
+        <plugin
+            filename="libignition-gazebo-multicopter-control-system.so"
             name="ignition::gazebo::systems::MulticopterVelocityControl">
-      <robotNamespace>X3</robotNamespace>
-      <comLinkName>base_link</comLinkName>
-      <velocityGain>2 2 2</velocityGain>
-      <attitudeGain>1.0 2.5 0.10</attitudeGain>
-      <angularRateGain>0.20 0.26 0.10</angularRateGain>
-      <maximumLinearAcceleration>2 2 2</maximumLinearAcceleration>
-      <cmd_vel_topic>cmd_vel</cmd_vel_topic>
-      <motor_velocity_command_topic>gazebo/command/motor_speed</motor_velocity_command_topic>
-      <rotorConfiguration>
-        <rotor><jointName>rotor_0_joint</jointName><linkName>rotor_0</linkName><direction> 1</direction><forceConstant>8.54858e-06</forceConstant><momentConstant>0.016</momentConstant></rotor>
-        <rotor><jointName>rotor_1_joint</jointName><linkName>rotor_1</linkName><direction> 1</direction><forceConstant>8.54858e-06</forceConstant><momentConstant>0.016</momentConstant></rotor>
-        <rotor><jointName>rotor_2_joint</jointName><linkName>rotor_2</linkName><direction>-1</direction><forceConstant>8.54858e-06</forceConstant><momentConstant>0.016</momentConstant></rotor>
-        <rotor><jointName>rotor_3_joint</jointName><linkName>rotor_3</linkName><direction>-1</direction><forceConstant>8.54858e-06</forceConstant><momentConstant>0.016</momentConstant></rotor>
-      </rotorConfiguration>
-    </plugin>
-  </gazebo>
-  <!-- Sensors system -->
-  <gazebo>
-    <plugin filename="libignition-gazebo-sensors-system.so"
-            name="ignition::gazebo::systems::Sensors"/>
-  </gazebo>
-  <!-- LiDAR (unchanged) -->
-  <gazebo reference="base_scan">
-    <material>Gazebo/FlatBlack</material>
-    <sensor type="gpu_lidar" name="lidar">
-      <pose relative_to='base_scan'>0 0 0 0 0 0</pose>
-      <visualize>$(arg laser_visual)</visualize>
-      <topic>X3/scan</topic>
-      <update_rate>10</update_rate>
-      <gz_frame_id>base_scan</gz_frame_id>
-      <ray>
-        <scan>
-          <horizontal><samples>360</samples><resolution>1</resolution><min_angle>0.0</min_angle><max_angle>6.28319</max_angle></horizontal>
-          <vertical><samples>64</samples><resolution>1</resolution><min_angle>-0.2618</min_angle><max_angle>0.2618</max_angle></vertical>
-        </scan>
-        <range><min>0.4</min><max>40</max><resolution>0.015</resolution></range>
-        <noise><type>gaussian</type><mean>0.0</mean><stddev>0.01</stddev></noise>
-      </ray>
-      <always_on>true</always_on>
-    </sensor>
-  </gazebo>
-  <!-- ===== RGB CAMERA ===== -->
-  <gazebo reference="rgbd_camera_link">
-    <sensor name="rgb_camera" type="camera">
-      <pose relative_to="rgbd_camera_link">0 0 0 0 0 0</pose>
-      <visualize>$(arg camera_visual)</visualize>
-      <topic>X3/rgbd_camera/image</topic>
-      <update_rate>30</update_rate>
-      <gz_frame_id>rgbd_camera_optical_frame</gz_frame_id>
-      <camera>
-        <horizontal_fov>1.047</horizontal_fov>                <!-- ~60 deg -->
-        <image><width>640</width><height>480</height><format>R8G8B8</format></image>
-        <clip><near>0.1</near><far>100</far></clip>
-      </camera>
-      <!-- Camera info is published automatically by Ignition camera -->
-    </sensor>
-  </gazebo>
-  <!-- ===== DEPTH CAMERA ===== -->
-  <gazebo reference="rgbd_camera_link">
-    <sensor name="depth_camera" type="depth_camera">
-      <pose relative_to="rgbd_camera_link">0 0 0 0 0 0</pose>
-      <visualize>$(arg depth_visual)</visualize>
-      <topic>X3/rgbd_camera/depth_image</topic>
-      <update_rate>30</update_rate>
-      <gz_frame_id>rgbd_camera_optical_frame</gz_frame_id>
-      <camera>
-        <horizontal_fov>1.047</horizontal_fov>
-        <image>
-          <width>640</width>
-          <height>480</height>
-          <!-- Use L16 so bridging to ROS Depth (16UC1) & depthimage_to_laserscan is easy -->
-          <format>L16</format>
-        </image>
-        <clip><near>0.2</near><far>20.0</far></clip>
-      </camera>
-    </sensor>
-  </gazebo>
-  <!-- IMU -->
-  <gazebo reference="imu_link">
-    <sensor type="imu" name="imu">
-      <always_on>true</always_on>
-      <visualize>$(arg imu_visual)</visualize>
-      <update_rate>100</update_rate>
-      <topic>X3/imu</topic>
-      <gz_frame_id>imu_link</gz_frame_id>
-      <imu>
-        <angular_velocity>
-          <x><noise type="gaussian"><mean>0.0</mean><stddev>2e-4</stddev><bias_mean>0.0000075</bias_mean><bias_stddev>0.0000008</bias_stddev></noise></x>
-          <y><noise type="gaussian"><mean>0.0</mean><stddev>2e-4</stddev><bias_mean>0.0000075</bias_mean><bias_stddev>0.0000008</bias_stddev></noise></y>
-          <z><noise type="gaussian"><mean>0.0</mean><stddev>2e-4</stddev><bias_mean>0.0000075</bias_mean><bias_stddev>0.0000008</bias_stddev></noise></z>
-        </angular_velocity>
-        <linear_acceleration>
-          <x><noise type="gaussian"><mean>0.0</mean><stddev>1.7e-2</stddev><bias_mean>0.1</bias_mean><bias_stddev>0.001</bias_stddev></noise></x>
-          <y><noise type="gaussian"><mean>0.0</mean><stddev>1.7e-2</stddev><bias_mean>0.1</bias_mean><bias_stddev>0.001</bias_stddev></noise></y>
-          <z><noise type="gaussian"><mean>0.0</mean><stddev>1.7e-2</stddev><bias_mean>0.1</bias_mean><bias_stddev>0.001</bias_stddev></noise></z>
-        </linear_acceleration>
-      </imu>
-      <plugin filename="ignition-gazebo-imu-system"
-              name="ignition::gazebo::systems::Imu"/>
-    </sensor>
-    <material>Gazebo/Grey</material>
-  </gazebo>
-  <!-- Odometry & joint states (unchanged) -->
-  <gazebo>
-    <plugin filename="ignition-gazebo-odometry-publisher-system"
+            <robotNamespace>X3</robotNamespace>
+            <comLinkName>base_link</comLinkName>
+            <velocityGain>2 2 2</velocityGain>
+            <attitudeGain>1.0 2.5 0.10</attitudeGain>
+            <angularRateGain>0.20 0.26 0.10</angularRateGain>
+            <maximumLinearAcceleration>2 2 2</maximumLinearAcceleration>
+            <cmd_vel_topic>cmd_vel</cmd_vel_topic>
+            <motor_velocity_command_topic>gazebo/command/motor_speed</motor_velocity_command_topic>
+            <rotorConfiguration>
+                <rotor>
+                    <jointName>rotor_0_joint</jointName>
+                    <linkName>rotor_0</linkName>
+                    <direction>1</direction>
+                    <forceConstant>8.54858e-06</forceConstant>
+                    <momentConstant>0.016</momentConstant>
+                </rotor>
+                <rotor>
+                    <jointName>rotor_1_joint</jointName>
+                    <linkName>rotor_1</linkName>
+                    <direction>1</direction>
+                    <forceConstant>8.54858e-06</forceConstant>
+                    <momentConstant>0.016</momentConstant>
+                </rotor>
+                <rotor>
+                    <jointName>rotor_2_joint</jointName>
+                    <linkName>rotor_2</linkName>
+                    <direction>-1</direction>
+                    <forceConstant>8.54858e-06</forceConstant>
+                    <momentConstant>0.016</momentConstant>
+                </rotor>
+                <rotor>
+                    <jointName>rotor_3_joint</jointName>
+                    <linkName>rotor_3</linkName>
+                    <direction>-1</direction>
+                    <forceConstant>8.54858e-06</forceConstant>
+                    <momentConstant>0.016</momentConstant>
+                </rotor>
+            </rotorConfiguration>
+        </plugin>
+        <!-- RGB camera angle -->
+        <plugin
+            filename="libignition-gazebo-joint-position-controller-system.so"
+            name="ignition::gazebo::systems::JointPositionController">
+            <joint_name>rgb_camera_joint</joint_name>
+            <topic>X3/rgb_camera/angle</topic>
+            <p_gain>1</p_gain>
+            <i_gain>0.1</i_gain>
+            <d_gain>0.01</d_gain>
+            <i_max>1</i_max>
+            <i_min>-1</i_min>
+            <cmd_max>1000</cmd_max>
+            <cmd_min>-1000</cmd_min>
+        </plugin>
+    </gazebo>
+    <!-- Sensors plugin for LiDAR -->
+    <gazebo>
+        <plugin
+            filename="libignition-gazebo-sensors-system.so"
+            name="ignition::gazebo::systems::Sensors">
+        </plugin>
+    </gazebo>
+    <!-- LiDAR -->
+    <gazebo reference="base_scan">
+        <material>Gazebo/FlatBlack</material>
+        <sensor type="gpu_lidar" name="lidar">
+            <pose relative_to='base_scan'>0 0 0 0 0 0</pose>
+            <visualize>$(arg laser_visual)</visualize>
+            <topic>X3/scan</topic>
+            <update_rate>10</update_rate>
+            <gz_frame_id>base_scan</gz_frame_id>
+            <ray>
+                <scan>
+                    <horizontal>
+                        <samples>360</samples>
+                        <resolution>1</resolution>
+                        <min_angle>0.0</min_angle>
+                        <max_angle>6.28319</max_angle>
+                    </horizontal>
+                    <vertical>
+                        <samples>64</samples>
+                        <resolution>1</resolution>
+                        <min_angle>-0.2618</min_angle> <!-- ~ 15 deg -->
+                        <max_angle>0.2618</max_angle>
+                    </vertical>
+                </scan>
+                <range>
+                    <min>0.4</min>
+                    <max>40</max>
+                    <resolution>0.015</resolution>
+                </range>
+                <noise>
+                    <type>gaussian</type>
+                    <mean>0.0</mean>
+                    <stddev>0.01</stddev>
+                </noise>
+            </ray>
+            <always_on>true</always_on>
+        </sensor>
+    </gazebo>
+    <!-- ===== RGB CAMERA ===== -->
+    <gazebo reference="rgbd_camera_link">
+      <sensor name="rgb_camera" type="camera">
+        <pose relative_to="rgbd_camera_link">0 0 0 0 0 0</pose>
+        <visualize>$(arg camera_visual)</visualize>
+        <topic>X3/rgbd_camera/image</topic>
+        <update_rate>30</update_rate>
+        <gz_frame_id>rgbd_camera_optical_frame</gz_frame_id>
+        <camera>
+          <horizontal_fov>1.047</horizontal_fov>                <!-- ~60 deg -->
+          <image><width>640</width><height>480</height><format>R8G8B8</format></image>
+          <clip><near>0.1</near><far>100</far></clip>
+        </camera>
+        <!-- Camera info is published automatically by Ignition camera -->
+      </sensor>
+    </gazebo>
+    <!-- ===== DEPTH CAMERA ===== -->
+    <gazebo reference="rgbd_camera_link">
+      <sensor name="depth_camera" type="depth_camera">
+        <pose relative_to="rgbd_camera_link">0 0 0 0 0 0</pose>
+        <visualize>$(arg depth_visual)</visualize>
+        <topic>X3/rgbd_camera/depth_image</topic>
+        <update_rate>30</update_rate>
+        <gz_frame_id>rgbd_camera_optical_frame</gz_frame_id>
+        <camera>
+          <horizontal_fov>1.047</horizontal_fov>
+          <image>
+            <width>640</width>
+            <height>480</height>
+            <!-- Use L16 so bridging to ROS Depth (16UC1) & depthimage_to_laserscan is easy -->
+            <format>L16</format>
+          </image>
+          <clip><near>0.2</near><far>20.0</far></clip>
+        </camera>
+      </sensor>
+    </gazebo>
+    <!-- IMU Sensor -->
+    <gazebo reference="imu_link">
+        <sensor type="imu" name="imu">
+            <always_on>true</always_on>
+            <visualize>$(arg imu_visual)</visualize>
+            <update_rate>100</update_rate>
+            <topic>X3/imu</topic>
+            <gz_frame_id>imu_link</gz_frame_id>
+            <imu>
+                <angular_velocity>
+                    <x>
+                        <noise type="gaussian">
+                            <mean>0.0</mean>
+                            <stddev>2e-4</stddev>
+                            <bias_mean>0.0000075</bias_mean>
+                            <bias_stddev>0.0000008</bias_stddev>
+                        </noise>
+                    </x>
+                    <y>
+                        <noise type="gaussian">
+                            <mean>0.0</mean>
+                            <stddev>2e-4</stddev>
+                            <bias_mean>0.0000075</bias_mean>
+                            <bias_stddev>0.0000008</bias_stddev>
+                        </noise>
+                    </y>
+                    <z>
+                        <noise type="gaussian">
+                            <mean>0.0</mean>
+                            <stddev>2e-4</stddev>
+                            <bias_mean>0.0000075</bias_mean>
+                            <bias_stddev>0.0000008</bias_stddev>
+                        </noise>
+                    </z>
+                </angular_velocity>
+                <linear_acceleration>
+                    <x>
+                        <noise type="gaussian">
+                            <mean>0.0</mean>
+                            <stddev>1.7e-2</stddev>
+                            <bias_mean>0.1</bias_mean>
+                            <bias_stddev>0.001</bias_stddev>
+                        </noise>
+                    </x>
+                    <y>
+                        <noise type="gaussian">
+                            <mean>0.0</mean>
+                            <stddev>1.7e-2</stddev>
+                            <bias_mean>0.1</bias_mean>
+                            <bias_stddev>0.001</bias_stddev>
+                        </noise>
+                    </y>
+                    <z>
+                        <noise type="gaussian">
+                            <mean>0.0</mean>
+                            <stddev>1.7e-2</stddev>
+                            <bias_mean>0.1</bias_mean>
+                            <bias_stddev>0.001</bias_stddev>
+                        </noise>
+                    </z>
+                </linear_acceleration>
+            </imu>
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